File: JEGGER_s-link.sch (KiCad schematic (older format))
At the start: 40 parts, among them J1 USB, J2 TC, J3 PINH, J4 RX, J5 TX, P1 STM, Q1 S9013, U1 USBLC6-4, U2 MCP1700T-3302E/TT, U3 STM32F103CBTx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

Commit message: updated files
Parts:
- removed R10, R9: 100, otter:R_0402, symbol Device:R_Small
- added R? (x2): 5k1, otter:R_0402, symbol Device:R_Small
- added R?: 1k5, otter:R_0402, symbol Device:R_Small
- R3: value 3k3 -> 5k1
Connections:
- net D+: now also R?.2; no longer Q1.2 (E)
- net GND: now also Y1.2, Y1.4; no longer Y1.1, Y1.3
- net LED_STLINK: now also R?.1, R?.2
- net at C4.2, U3.5 (PD0): now also Y1.1; no longer Y1.2
- net at C5.1, U3.6 (PD1): now also Y1.3; no longer Y1.4
- net at D4.2 (A): now also R?.1
- net at D3.1 (K): now also R?.2
- new net: Q1.2 (E), R?.1
Other:
- moved on the sheet: C4, C5
Changed lines of the file:
@@
 	7800 3100 8000 3100
-$Comp
-L power:GND #PWR0114
-U 1 1 5E7C39CC
-P 7350 3000
-F 0 "#PWR0114" H 7350 2750 50  0001 C CNN
-F 1 "GND" V 7355 2872 50  0000 R CNN
-F 2 "" H 7350 3000 50  0001 C CNN
-F 3 "" H 7350 3000 50  0001 C CNN
-	1    7350 3000
-	0    1    1    0
-$EndComp
-$Comp
-L Device:C_Small C5
-U 1 1 5E7C58F5
-P 7400 3250
-F 0 "C5" V 7537 3250 50  0000 C CNN
-F 1 "22p" V 7628 3250 50  0000 C CNN
-F 2 "otter:C_0402" H 7400 3250 50  0001 C CNN
-F 3 "~" H 7400 3250 50  0001 C CNN
-	1    7400 3250
-	0    1    1    0
-$EndComp
-$Comp
-L Device:C_Small C4
-U 1 1 5E7C6116
-P 7400 2750
-F 0 "C4" V 7629 2750 50  0000 C CNN
-F 1 "22p" V 7538 2750 50  0000 C CNN
-F 2 "otter:C_0402" H 7400 2750 50  0001 C CNN
-F 3 "~" H 7400 2750 50  0001 C CNN
-	1    7400 2750
-	0    -1   -1   0
-$EndComp
-$Comp
-L power:GND #PWR0115
-U 1 1 5E7C9132
-P 7300 2750
-F 0 "#PWR0115" H 7300 2500 50  0001 C CNN
-F 1 "GND" V 7305 2622 50  0000 R CNN
-F 2 "" H 7300 2750 50  0001 C CNN
-F 3 "" H 7300 2750 50  0001 C CNN
-	1    7300 2750
-	0    1    1    0
-$EndComp
-$Comp
-L power:GND #PWR0116
-U 1 1 5E7C9A53
-P 7300 3250
-F 0 "#PWR0116" H 7300 3000 50  0001 C CNN
-F 1 "GND" V 7305 3122 50  0000 R CNN
-F 2 "" H 7300 3250 50  0001 C CNN
-F 3 "" H 7300 3250 50  0001 C CNN
-	1    7300 3250
-	0    1    1    0
-$EndComp
 $Comp
 L otter:USBLC6-4 U1
@@
 P 3700 4450
 F 0 "R3" H 3641 4496 50  0000 R CNN
-F 1 "3k3" H 3641 4405 50  0000 R CNN
+F 1 "5k1" H 3641 4405 50  0000 R CNN
 F 2 "otter:R_0402" H 3700 4450 50  0001 C CNN
 F 3 "~" H 3700 4450 50  0001 C CNN
@@
 	1    0    0    -1
 $EndComp
-$Comp
-L Device:Crystal_GND24 Y1
-U 1 1 5E87D1F2
-P 7500 3000
-F 0 "Y1" H 7750 2550 50  0000 L CNN
-F 1 "8Mhz" H 7650 2650 50  0000 L CNN
-F 2 "Crystal:Crystal_SMD_3225-4Pin_3.2x2.5mm" H 7500 3000 50  0001 C CNN
-F 3 "~" H 7500 3000 50  0001 C CNN
-	1    7500 3000
-	1    0    0    -1
-$EndComp
-Wire Wire Line
-	7500 3250 7800 3250
-Wire Wire Line
-	7800 2750 7500 2750
-Wire Wire Line
-	7800 2750 7800 2900
-Wire Wire Line
-	7800 3100 7800 3250
-$Comp
-L power:GND #PWR0124
-U 1 1 5E887A23
-P 7650 3000
-F 0 "#PWR0124" H 7650 2750 50  0001 C CNN
-F 1 "GND" V 7655 2872 50  0000 R CNN
-F 2 "" H 7650 3000 50  0001 C CNN
-F 3 "" H 7650 3000 50  0001 C CNN
-	1    7650 3000
-	0    -1   -1   0
-$EndComp
-Wire Wire Line
-	7500 2800 7500 2750
-Connection ~ 7500 2750
-Wire Wire Line
-	7500 3200 7500 3250
-Connection ~ 7500 3250
 $Comp
 L MCU_ST_STM32F1:STM32F103CBTx U3
@@
 $EndComp
 $Comp
-L Device:R_Small R10
-U 1 1 5E8367B2
-P 5750 7050
-F 0 "R10" V 5854 7050 50  0000 C CNN
-F 1 "100" V 5945 7050 50  0000 C CNN
-F 2 "otter:R_0402" H 5750 7050 50  0001 C CNN
-F 3 "~" H 5750 7050 50  0001 C CNN
-	1    5750 7050
-	0    1    1    0
-$EndComp
-$Comp
 L power:GND #PWR0141
 U 1 1 5E8367B8
@@
 	-1   0    0    1
 $EndComp
-$Comp
-L Device:R_Small R9
-U 1 1 5E838BCE
-P 5750 6850
-F 0 "R9" V 5946 6850 50  0000 C CNN
-F 1 "100" V 5855 6850 50  0000 C CNN
-F 2 "otter:R_0402" H 5750 6850 50  0001 C CNN
-F 3 "~" H 5750 6850 50  0001 C CNN
-	1    5750 6850
-	0    -1   -1   0
-$EndComp
 Wire Wire Line
 	6250 7050 5950 7050
@@
 	1    0    0    -1
 $EndComp
-Text GLabel 6050 5900 3    50   Input ~ 0
+Text GLabel 6050 6200 3    50   Input ~ 0
 D+
 $Comp
@@
 	-1   0    0    1
 $EndComp
+$Comp
+L power:GND #PWR0114
+U 1 1 5E7C39CC
+P 7300 3000
+F 0 "#PWR0114" H 7300 2750 50  0001 C CNN
+F 1 "GND" V 7305 2872 50  0000 R CNN
+F 2 "" H 7300 3000 50  0001 C CNN
+F 3 "" H 7300 3000 50  0001 C CNN
+	1    7300 3000
+	0    1    1    0
+$EndComp
+$Comp
+L power:GND #PWR0124
+U 1 1 5E887A23
+P 7700 3000
+F 0 "#PWR0124" H 7700 2750 50  0001 C CNN
+F 1 "GND" V 7705 2872 50  0000 R CNN
+F 2 "" H 7700 3000 50  0001 C CNN
+F 3 "" H 7700 3000 50  0001 C CNN
+	1    7700 3000
+	0    -1   -1   0
+$EndComp
+$Comp
+L Device:C_Small C4
+U 1 1 5E7C6116
+P 7400 2800
+F 0 "C4" V 7629 2800 50  0000 C CNN
+F 1 "22p" V 7538 2800 50  0000 C CNN
+F 2 "otter:C_0402" H 7400 2800 50  0001 C CNN
+F 3 "~" H 7400 2800 50  0001 C CNN
+	1    7400 2800
+	0    -1   -1   0
+$EndComp
+$Comp
+L power:GND #PWR0115
+U 1 1 5E7C9132
+P 7300 2800
+F 0 "#PWR0115" H 7300 2550 50  0001 C CNN
+F 1 "GND" V 7305 2672 50  0000 R CNN
+F 2 "" H 7300 2800 50  0001 C CNN
+F 3 "" H 7300 2800 50  0001 C CNN
+	1    7300 2800
+	0    1    1    0
+$EndComp
+Wire Wire Line
+	7800 2800 7500 2800
+Wire Wire Line
+	7500 2850 7500 2800
+Connection ~ 7500 2800
+Wire Wire Line
+	7800 2800 7800 2900
+$Comp
+L Device:C_Small C5
+U 1 1 5E7C58F5
+P 7400 3200
+F 0 "C5" V 7537 3200 50  0000 C CNN
+F 1 "22p" V 7628 3200 50  0000 C CNN
+F 2 "otter:C_0402" H 7400 3200 50  0001 C CNN
+F 3 "~" H 7400 3200 50  0001 C CNN
+	1    7400 3200
+	0    1    1    0
+$EndComp
+$Comp
+L power:GND #PWR0116
+U 1 1 5E7C9A53
+P 7300 3200
+F 0 "#PWR0116" H 7300 2950 50  0001 C CNN
+F 1 "GND" V 7305 3072 50  0000 R CNN
+F 2 "" H 7300 3200 50  0001 C CNN
+F 3 "" H 7300 3200 50  0001 C CNN
+	1    7300 3200
+	0    1    1    0
+$EndComp
+Wire Wire Line
+	7500 3200 7800 3200
+Wire Wire Line
+	7500 3150 7500 3200
+Connection ~ 7500 3200
+Wire Wire Line
+	7800 3100 7800 3200
+$Comp
+L Device:Crystal_GND24 Y1
+U 1 1 5E87D1F2
+P 7500 3000
+F 0 "Y1" V 7150 3150 50  0000 L CNN
+F 1 "8Mhz" V 7250 3100 50  0000 L CNN
+F 2 "Crystal:Crystal_SMD_3225-4Pin_3.2x2.5mm" H 7500 3000 50  0001 C CNN
+F 3 "~" H 7500 3000 50  0001 C CNN
+	1    7500 3000
+	0    1    1    0
+$EndComp
+$Comp
+L Device:R_Small R?
+U 1 1 5E888CC5
+P 5750 7050
+F 0 "R?" V 5646 7050 50  0000 C CNN
+F 1 "5k1" V 5555 7050 50  0000 C CNN
+F 2 "otter:R_0402" H 5750 7050 50  0001 C CNN
+F 3 "~" H 5750 7050 50  0001 C CNN
+	1    5750 7050
+	0    -1   -1   0
+$EndComp
+$Comp
+L Device:R_Small R?
+U 1 1 5E88A4FF
+P 5750 6850
+F 0 "R?" V 5554 6850 50  0000 C CNN
+F 1 "5k1" V 5645 6850 50  0000 C CNN
+F 2 "otter:R_0402" H 5750 6850 50  0001 C CNN
+F 3 "~" H 5750 6850 50  0001 C CNN
+	1    5750 6850
+	0    1    1    0
+$EndComp
+$Comp
+L Device:R_Small R?
+U 1 1 5E8932E2
+P 6050 6050
+F 0 "R?" V 6246 6050 50  0000 C CNN
+F 1 "1k5" V 6155 6050 50  0000 C CNN
+F 2 "otter:R_0402" H 6050 6050 50  0001 C CNN
+F 3 "~" H 6050 6050 50  0001 C CNN
+	1    6050 6050
+	1    0    0    -1
+$EndComp
+Wire Wire Line
+	6050 5950 6050 5900
+Wire Wire Line
+	6050 6200 6050 6150
 $EndSCHEMATC

Commit message: push
Parts:
- removed Q1: S9013, Package_TO_SOT_SMD:SOT-23, symbol Transistor_BJT:BC817
- removed R6: 100, otter:R_0402, symbol Device:R_Small
- removed R7: 10k, otter:R_0402, symbol Device:R_Small
- removed R8: 36k, otter:R_0402, symbol Device:R_Small
- gave numbers to parts that had none: 3
Connections:
- net +3V3: now also R11.1
Changed lines of the file:
@@
-	1    0    0    -1
-$EndComp
-$Comp
-L Transistor_BJT:BC817 Q1
-U 1 1 5E859BBA
-P 5950 5700
-F 0 "Q1" H 6140 5746 50  0000 L CNN
-F 1 "S9013" H 6140 5655 50  0000 L CNN
-F 2 "Package_TO_SOT_SMD:SOT-23" H 6150 5625 50  0001 L CIN
-F 3 "http://www.fairchildsemi.com/ds/BC/BC817.pdf" H 5950 5700 50  0001 L CNN
-	1    5950 5700
 	1    0    0    -1
 $EndComp
@@
 D+
 $Comp
-L Device:R_Small R6
-U 1 1 5E868219
-P 5400 5700
-F 0 "R6" V 5596 5700 50  0000 C CNN
-F 1 "100" V 5505 5700 50  0000 C CNN
-F 2 "otter:R_0402" H 5400 5700 50  0001 C CNN
-F 3 "~" H 5400 5700 50  0001 C CNN
-	1    5400 5700
-	0    -1   -1   0
-$EndComp
-$Comp
 L power:+3.3V #PWR0144
 U 1 1 5E86821F
-P 6050 5500
-F 0 "#PWR0144" H 6050 5350 50  0001 C CNN
-F 1 "+3.3V" H 6065 5673 50  0000 C CNN
-F 2 "" H 6050 5500 50  0001 C CNN
-F 3 "" H 6050 5500 50  0001 C CNN
-	1    6050 5500
-	1    0    0    -1
-$EndComp
-$Comp
-L Device:R_Small R7
-U 1 1 5E873E28
-P 5650 5500
-F 0 "R7" H 5591 5454 50  0000 R CNN
-F 1 "10k" H 5591 5545 50  0000 R CNN
-F 2 "otter:R_0402" H 5650 5500 50  0001 C CNN
-F 3 "~" H 5650 5500 50  0001 C CNN
-	1    5650 5500
-	-1   0    0    1
-$EndComp
-$Comp
-L Device:R_Small R8
-U 1 1 5E87543F
-P 5650 5900
-F 0 "R8" H 5709 5854 50  0000 L CNN
-F 1 "36k" H 5709 5945 50  0000 L CNN
-F 2 "otter:R_0402" H 5650 5900 50  0001 C CNN
-F 3 "~" H 5650 5900 50  0001 C CNN
-	1    5650 5900
-	-1   0    0    1
-$EndComp
-Wire Wire Line
-	5650 5800 5650 5700
-Wire Wire Line
-	5650 5700 5750 5700
-Wire Wire Line
-	5650 5600 5650 5700
-Connection ~ 5650 5700
-Wire Wire Line
-	5650 5700 5500 5700
-$Comp
-L power:GND #PWR0145
-U 1 1 5E87C1A9
-P 5650 6000
-F 0 "#PWR0145" H 5650 5750 50  0001 C CNN
-F 1 "GND" H 5655 5827 50  0000 C CNN
-F 2 "" H 5650 6000 50  0001 C CNN
-F 3 "" H 5650 6000 50  0001 C CNN
-	1    5650 6000
-	1    0    0    -1
-$EndComp
-Text GLabel 5300 5700 0    50   Input ~ 0
-USB_RENUM
-$Comp
-L power:VBUS #PWR0146
-U 1 1 5E88C00E
-P 5650 5400
-F 0 "#PWR0146" H 5650 5250 50  0001 C CNN
-F 1 "VBUS" V 5665 5528 50  0000 L CNN
-F 2 "" H 5650 5400 50  0001 C CNN
-F 3 "" H 5650 5400 50  0001 C CNN
-	1    5650 5400
+P 6050 5900
+F 0 "#PWR0144" H 6050 5750 50  0001 C CNN
+F 1 "+3.3V" H 6065 6073 50  0000 C CNN
+F 2 "" H 6050 5900 50  0001 C CNN
+F 3 "" H 6050 5900 50  0001 C CNN
+	1    6050 5900
 	1    0    0    -1
 $EndComp
@@
 $EndComp
 $Comp
-L Device:R_Small R?
+L Device:R_Small R10
 U 1 1 5E888CC5
 P 5750 7050
-F 0 "R?" V 5646 7050 50  0000 C CNN
+F 0 "R10" V 5646 7050 50  0000 C CNN
 F 1 "5k1" V 5555 7050 50  0000 C CNN
 F 2 "otter:R_0402" H 5750 7050 50  0001 C CNN
@@
 $EndComp
 $Comp
-L Device:R_Small R?
+L Device:R_Small R9
 U 1 1 5E88A4FF
 P 5750 6850
-F 0 "R?" V 5554 6850 50  0000 C CNN
+F 0 "R9" V 5554 6850 50  0000 C CNN
 F 1 "5k1" V 5645 6850 50  0000 C CNN
 F 2 "otter:R_0402" H 5750 6850 50  0001 C CNN
@@
 $EndComp
 $Comp
-L Device:R_Small R?
+L Device:R_Small R11
 U 1 1 5E8932E2
 P 6050 6050
-F 0 "R?" V 6246 6050 50  0000 C CNN
+F 0 "R11" V 6246 6050 50  0000 C CNN
 F 1 "1k5" V 6155 6050 50  0000 C CNN
 F 2 "otter:R_0402" H 6050 6050 50  0001 C CNN

Commit message: push
Parts:
- D2: symbol Diode:BAT60A -> JEGGER_s-link-rescue:BAT60A-Diode
Other:
- moved on the sheet: C10, C11, C2, C3, D1, D2, D3, D4, J1, J2, J3, J4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
