File: JEGGER_s-link.kicad_pcb (KiCad board)
At the start: 2 copper layers, 37.6 x 16.1 mm, 42 parts, among them J1 USB, J2 TC, J3 PINH, J4 RX, J5 TX, P1 STM, Q1 S9013, U1 USBLC6-4, U2 MCP1700T-3302E/TT, U3 STM32F103CBTx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

Commit message: updated files
Parts:
- added R11: 1k5, otter:R_0402, F.Cu at (123.0, 91.0)
- R10, R9: value 100 -> 5k1
- R3: value 3k3 -> 5k1
- moved R9 0.80 mm to (123.8, 96.2), turned to 0 degrees
- turned R10 to 180 degrees
- turned C4 to 225 degrees
- turned C5 to 225 degrees
- turned Y1 to 315 degrees
Connections:
- Q1 pad 2: D+ -> Net-(Q1-Pad2)
- R10 pad 1: LED_STLINK -> Net-(D4-Pad2)
- R10 pad 2: Net-(D4-Pad2) -> LED_STLINK
- R9 pad 1: Net-(D3-Pad1) -> LED_STLINK
- R9 pad 2: LED_STLINK -> Net-(D3-Pad1)
- Y1 pad 1: GND -> Net-(C4-Pad2)
- Y1 pad 2: Net-(C4-Pad2) -> GND
- Y1 pad 3: GND -> Net-(C5-Pad1)
- Y1 pad 4: Net-(C5-Pad1) -> GND
Routing:
- net GND: track 38.6 -> 34.3 mm
- net Net-(C5-Pad1): track 6.39 -> 3.53 mm
- net Net-(C4-Pad2): track 4.85 -> 6.09 mm

Commit message: push
Parts:
- removed Q1: S9013, Package_TO_SOT_SMD:SOT-23
- removed R6: 100, otter:R_0402
- removed R7: 10k, otter:R_0402
- removed R8: 36k, otter:R_0402
- moved R11 3.87 mm to (120.9, 94.3), turned to 315 degrees
- moved R9 1.64 mm to (122.4, 95.4), turned to 90 degrees
- moved R10 0.31 mm to (123.6, 96.7)
Connections:
- R11 pad 1: Net-(Q1-Pad2) -> +3V3
Routing:
- net Net-(Q1-Pad1): track 8.15 -> 0.00 mm
- net VBUS: track 23.7 -> 18.5 mm
- net Net-(D3-Pad1): track 15.7 -> 18.9 mm
- net USB_RENUM: track 2.41 -> 0.00 mm
- net +3V3: track 54.3 -> 52.9 mm

Commit message: updated to KiCAD 6
Other:
- net class Default removed
- board text added: "Design by: @_Jana_Marie"
- board text removed: "Design by: @JanHenrikH"
